File: Hardware/LED-RingCoder.sch (EAGLE design)
At the start: 37 parts, among them IC1 74LS595D, IC2 74LS595D, U1 ENCODER_RGB

Commit message: Adding EN/GND and CLR/VCC jumpers
Parts:
- added JP10, JP7: (no value), SparkFun-Passives:JUMPER-2SMD-NC
Connections:
- net CLEAR: now also JP10.2
- net EN: now also JP7.2
- net GND: now also JP7.1
- net VCC: now also JP10.1
Other:
- moved on the sheet: LED1, R17, R18, R19, R20, U1
